Commit message: Final commit

File: snatcher/urdf/snatcher.gazebo.xacro (robot description, xacro)
@@ -5,5 +5,5 @@
   <xacro:arg name="imu_visual"    default="false"/>
   <gazebo reference="base_link">
-    <material>Gazebo/DarkGrey</material>
+    <material>Gazebo/Turquoise </material>
   </gazebo>
   <gazebo reference="wheel_left_link">

File: snatcher/urdf/snatcher.rviz.xacro (robot description, xacro)
@@ -1,6 +1,6 @@
 <?xml version="1.0" ?>
 <robot name="myrover" xmlns:xacro="http://ros.org/wiki/xacro">
-  <xacro:include filename="$(find rover)/urdf/colors.xacro"/>
-  <xacro:include filename="$(find rover)/urdf/myrover.gazebo.xacro"/>
+  <xacro:include filename="$(find snatcher)/urdf/colors.xacro"/>
+  <xacro:include filename="$(find snatcher)/urdf/snatcher.gazebo.xacro"/>
   <link name="base_footprint"/>
   <joint name="base_joint" type="fixed">
@@ -70,5 +70,4 @@
       <origin xyz="0 0 0" rpy="0 0 0"/>
       <geometry>
-        <!--mesh filename="package://turtlebot3_description/meshes/wheels/left_tire.stl" scale="0.001 0.001 0.001"/-->
         <cylinder length="0.018" radius="0.06"/>
       </geometry>
@@ -99,5 +98,4 @@
       <origin xyz="0 0 0" rpy="0 0 0"/>
       <geometry>
-        <!--mesh filename="package://turtlebot3_description/meshes/wheels/right_tire.stl" scale="0.001 0.001 0.001"/-->
         <cylinder length="0.018" radius="0.06"/>
       </geometry>
@@ -174,5 +172,4 @@
       <origin xyz="0 0 0" rpy="0 0 0"/>
       <geometry>
-        <!--mesh filename="package://turtlebot3_description/meshes/sensors/lds.stl" scale="0.001 0.001 0.001"/-->
         <cylinder length="0.0315" radius="0.055"/>
       </geometry>
@@ -198,3 +195,63 @@
     <origin xyz="-0.064 0 0.35" rpy="0 0 0"/>
   </joint>
+<link name="left_door">
+		<visual>
+		  <origin xyz="0 -0.08 0" rpy="0 0 0"/>
+		  <geometry>
+		    <box size="0.01 0.15 0.3"/>
+		  </geometry>
+		  <material name="blue"/>
+		</visual>
+		<collision>
+		  <origin xyz="0 -0.08 0" rpy="0 0 0"/>
+		  <geometry>
+		    <box size="0.01 0.15 0.3"/>
+		  </geometry>
+		  <material name="blue"/>
+		</collision>
+		<inertial>
+		  <origin xyz="-0.1 -0.04 0" rpy="0 0 0"/>
+	    <mass value="0.1"/>
+	    <inertia ixx="0.035416666666667" ixy="0" ixz="0"
+	  		       iyy="0.035416666666667" iyz="0"
+		  	       izz="0.040833333333333" />
+    	</inertial>
+	</link>
+	<joint name="left_door_joint" type="revolute">
+	  <origin xyz="0.09 0.16 0.17" rpy="0 0 0" />
+		<parent link="base_link" />
+		<child link="left_door" />
+		<axis	xyz="0 0 1" />
+		<limit lower="0" upper="1.57" effort="2" velocity="2.0" />
+	</joint>
+	<link name="right_door">
+		<visual>
+		  <origin xyz="0 0.08 0" rpy="0 0 0"/>
+		  <geometry>
+		    <box size="0.01 0.15 0.3"/>
+		  </geometry>
+		  <material name="blue"/>
+		</visual>
+		<collision>
+		  <origin xyz="0 0.08 0" rpy="0 0 0"/>
+		  <geometry>
+		    <box size="0.01 0.15 0.3"/>
+		  </geometry>
+		  <material name="blue"/>
+		</collision>
+		<inertial>
+		  <origin xyz="-0.1 -0.04 0" rpy="0 0 0"/>
+	    <mass value="0.1"/>
+	    <inertia ixx="0.0002" ixy="0" ixz="0"
+	  		       iyy="0.0004" iyz="0"
+		  	       izz="0.0002" />
+    	</inertial>
+	</link>
+	<joint name="right_door_joint" type="revolute">
+	  <origin xyz="0.09 -0.16 0.17" rpy="0 0 0" />
+		<parent link="base_link" />
+		<child link="right_door" />
+		<axis	xyz="0 0 1" />
+		<limit lower="-1.57" upper="0" effort="2" velocity="2.0" />
+	</joint>
 </robot>
